Commit message: M03: Adding launch to display urdf and xacro model, pending explanations

File: m03_robot_description/m03_using_urdf/urdf/r2d2_model.urdf (robot description, URDF)
Before this commit: robot r2d2_urdf_mod, 39 links, 38 joints
Links:
- link left_gripper: geometry visual mesh filename=package://m03_using_urdf/meshes/l_finger.dae
- link left_tip: geometry visual mesh filename=package://m03_using_urdf/meshes/l_finger_tip.dae
- link right_gripper: geometry visual mesh filename=package://m03_using_urdf/meshes/l_finger.dae
- link right_tip: geometry visual mesh filename=package://m03_using_urdf/meshes/l_finger_tip.dae

File: m03_robot_description/m03_using_urdf/urdf/r2d2_model.urdf.xacro (robot description, xacro)
@@ -8,5 +8,6 @@
 <xacro:property name="baselen" value="0.4" />
 <xacro:property name="wheeldiam" value="0.07" />
-<xacro:property name="pi" value="3.1415" />
+<!-- PI is already defined in Python, which takes care of the calcs -->
+<!--xacro:property name="pi" value="3.1416" /-->
 <xacro:property name="shoulder" value="0.12"/>
 <xacro:property name="box" value="0.05"/>
@@ -196,10 +197,10 @@
         <origin rpy="${(reflect-1)/2*pi} 0 0" xyz="0 0 0"/>
         <geometry>
-        <mesh filename="package://urdf_tutorial/meshes/l_finger.dae"/>
-        </geometry>
-    </visual>
-    <collision>
-        <geometry>
-        <mesh filename="package://urdf_tutorial/meshes/l_finger.dae"/>
+        <mesh filename="package://m03_using_urdf/meshes/l_finger.dae"/>
+        </geometry>
+    </visual>
+    <collision>
+        <geometry>
+        <mesh filename="package://m03_using_urdf/meshes/l_finger.dae"/>
         </geometry>
         <origin rpy="${(reflect-1)/2*pi} 0 0" xyz="0 0 0"/>
@@ -215,10 +216,10 @@
         <origin rpy="${(reflect-1)/2*pi} 0 0" xyz="0.09137 0.00495 0"/>
         <geometry>
-        <mesh filename="package://urdf_tutorial/meshes/l_finger_tip.dae"/>
-        </geometry>
-    </visual>
-    <collision>
-        <geometry>
-        <mesh filename="package://urdf_tutorial/meshes/l_finger_tip.dae"/>
+        <mesh filename="package://m03_using_urdf/meshes/l_finger_tip.dae"/>
+        </geometry>
+    </visual>
+    <collision>
+        <geometry>
+        <mesh filename="package://m03_using_urdf/meshes/l_finger_tip.dae"/>
         </geometry>
         <origin rpy="${(reflect-1)/2*pi} 0 0" xyz="0.09137 0.00495 0"/>
